File: kicad_hiltop_loti_board/DigitalIO.sch (KiCad schematic (older format))
At the start: 36 parts

Commit message: Rev A
Parts:
- D14, D15, D16, D17, D18, D19, D20, D21, D22, D23, D24, D25, D26, D27, D28, D29, D30, D31: symbol Diode:BAV99 -> LoTI_Board-rescue:BAV99-Diode
- R125, R126, R127, R128, R129, R130, R131, R132, R133, R134, R135, R136, R137, R138, R139, R140, R141, R142: symbol device:R -> LoTI_Board-rescue:R-device
Changed lines of the file:
@@
 EESchema Schematic File Version 4
 LIBS:LoTI_Board-cache
-EELAYER 26 0
+EELAYER 29 0
 EELAYER END
 $Descr A3 16535 11693
@@
 	4000 3425 4000 3875
 $Comp
-L Diode:BAV99 D18
+L LoTI_Board-rescue:BAV99-Diode D18
 U 2 1 5C6F696C
 P 4200 3275
@@
 $EndComp
 $Comp
-L Diode:BAV99 D16
+L LoTI_Board-rescue:BAV99-Diode D16
 U 2 1 5C6F6973
 P 4000 3275
@@
 $EndComp
 $Comp
-L Diode:BAV99 D18
+L LoTI_Board-rescue:BAV99-Diode D18
 U 1 1 5C6F697A
 P 4250 5075
@@
 $EndComp
 $Comp
-L Diode:BAV99 D16
+L LoTI_Board-rescue:BAV99-Diode D16
 U 1 1 5C6F6981
 P 4050 5075
@@
 	3650 3675 3800 3675
 $Comp
-L device:R R125
+L LoTI_Board-rescue:R-device R125
 U 1 1 5C6F69A0
 P 3500 3675
@@
 $EndComp
 $Comp
-L Diode:BAV99 D14
+L LoTI_Board-rescue:BAV99-Diode D14
 U 1 1 5C6F69AD
 P 3850 5075
@@
 $EndComp
 $Comp
-L Diode:BAV99 D14
+L LoTI_Board-rescue:BAV99-Diode D14
 U 2 1 5C6F69B4
 P 3800 3275
@@
 Max 3mA per GPIO
 $Comp
-L device:R R126
+L LoTI_Board-rescue:R-device R126
 U 1 1 5C72D67A
 P 3500 3875
@@
 $EndComp
 $Comp
-L device:R R127
+L LoTI_Board-rescue:R-device R127
 U 1 1 5C72D782
 P 3500 4075
@@
 	3125 4275 3350 4275
 $Comp
-L device:R R128
+L LoTI_Board-rescue:R-device R128
 U 1 1 5C81CFA4
 P 3500 4275
@@
 	3125 4475 3350 4475
 $Comp
-L device:R R129
+L LoTI_Board-rescue:R-device R129
 U 1 1 5C875B29
 P 3500 4475
@@
 	3125 4675 3350 4675
 $Comp
-L device:R R130
+L LoTI_Board-rescue:R-device R130
 U 1 1 5C8CEAFE
 P 3500 4675
@@
 	3650 4675 4800 4675
 $Comp
-L Diode:BAV99 D20
+L LoTI_Board-rescue:BAV99-Diode D20
 U 1 1 5C8FC445
 P 4450 5075
@@
 $EndComp
 $Comp
-L Diode:BAV99 D22
+L LoTI_Board-rescue:BAV99-Diode D22
 U 1 1 5C8FC54D
 P 4650 5075
@@
 $EndComp
 $Comp
-L Diode:BAV99 D24
+L LoTI_Board-rescue:BAV99-Diode D24
 U 1 1 5C8FC667
 P 4850 5075
@@
 Connection ~ 4250 4075
 $Comp
-L Diode:BAV99 D20
+L LoTI_Board-rescue:BAV99-Diode D20
 U 2 1 5CAF93E8
 P 4400 3275
@@
 $EndComp
 $Comp
-L Diode:BAV99 D22
+L LoTI_Board-rescue:BAV99-Diode D22
 U 2 1 5CAF9502
 P 4600 3275
@@
 $EndComp
 $Comp
-L Diode:BAV99 D24
+L LoTI_Board-rescue:BAV99-Diode D24
 U 2 1 5CAF960E
 P 4800 3275
@@
 	4050 6775 4050 7225
 $Comp
-L Diode:BAV99 D19
+L LoTI_Board-rescue:BAV99-Diode D19
 U 2 1 5CCE0401
 P 4250 6625
@@
 $EndComp
 $Comp
-L Diode:BAV99 D17
+L LoTI_Board-rescue:BAV99-Diode D17
 U 2 1 5CCE0408
 P 4050 6625
@@
 $EndComp
 $Comp
-L Diode:BAV99 D19
+L LoTI_Board-rescue:BAV99-Diode D19
 U 1 1 5CCE040F
 P 4300 8425
@@
 $EndComp
 $Comp
-L Diode:BAV99 D17
+L LoTI_Board-rescue:BAV99-Diode D17
 U 1 1 5CCE0416
 P 4100 8425
@@
 	3700 7025 3850 7025
 $Comp
-L device:R R131
+L LoTI_Board-rescue:R-device R131
 U 1 1 5CCE0424
 P 3550 7025
@@
 $EndComp
 $Comp
-L Diode:BAV99 D15
+L LoTI_Board-rescue:BAV99-Diode D15
 U 1 1 5CCE0431
 P 3900 8425
@@
 $EndComp
 $Comp
-L Diode:BAV99 D15
+L LoTI_Board-rescue:BAV99-Diode D15
 U 2 1 5CCE0438
 P 3850 6625
@@
 	3175 7025 3400 7025
 $Comp
-L device:R R132
+L LoTI_Board-rescue:R-device R132
 U 1 1 5CCE0442
 P 3550 7225
@@
 $EndComp
 $Comp
-L device:R R133
+L LoTI_Board-rescue:R-device R133
 U 1 1 5CCE0449
 P 3550 7425
@@
 	3175 7625 3400 7625
 $Comp
-L device:R R134
+L LoTI_Board-rescue:R-device R134
 U 1 1 5CCE0460
 P 3550 7625
@@
 	3175 7825 3400 7825
 $Comp
-L device:R R135
+L LoTI_Board-rescue:R-device R135
 U 1 1 5CCE046B
 P 3550 7825
@@
 	3175 8025 3400 8025
 $Comp
-L device:R R136
+L LoTI_Board-rescue:R-device R136
 U 1 1 5CCE0476
 P 3550 8025
@@
 	3700 8025 4850 8025
 $Comp
-L Diode:BAV99 D21
+L LoTI_Board-rescue:BAV99-Diode D21
 U 1 1 5CCE0480
 P 4500 8425
@@
 $EndComp
 $Comp
-L Diode:BAV99 D23
+L LoTI_Board-rescue:BAV99-Diode D23
 U 1 1 5CCE0487
 P 4700 8425
@@
 $EndComp
 $Comp
-L Diode:BAV99 D25
+L LoTI_Board-rescue:BAV99-Diode D25
 U 1 1 5CCE048E
 P 4900 8425
@@
 	4300 7425 5925 7425
 $Comp
-L Diode:BAV99 D21
+L LoTI_Board-rescue:BAV99-Diode D21
 U 2 1 5CCE04B1
 P 4450 6625
@@
 $EndComp
 $Comp
-L Diode:BAV99 D23
+L LoTI_Board-rescue:BAV99-Diode D23
 U 2 1 5CCE04B8
 P 4650 6625
@@
 $EndComp
 $Comp
-L Diode:BAV99 D25
+L LoTI_Board-rescue:BAV99-Diode D25
 U 2 1 5CCE04BF
 P 4850 6625
@@
 	9500 3425 9500 3875
 $Comp
-L Diode:BAV99 D28
+L LoTI_Board-rescue:BAV99-Diode D28
 U 2 1 5E7ED93E
 P 9700 3275
@@
 $EndComp
 $Comp
-L Diode:BAV99 D27
+L LoTI_Board-rescue:BAV99-Diode D27
 U 2 1 5E7ED945
 P 9500 3275
@@
 $EndComp
 $Comp
-L Diode:BAV99 D28
+L LoTI_Board-rescue:BAV99-Diode D28
 U 1 1 5E7ED94C
 P 9750 5075
@@
 $EndComp
 $Comp
-L Diode:BAV99 D27
+L LoTI_Board-rescue:BAV99-Diode D27
 U 1 1 5E7ED953
 P 9550 5075
@@
 	9150 3675 9300 3675
 $Comp
-L device:R R137
+L LoTI_Board-rescue:R-device R137
 U 1 1 5E7ED961
 P 9000 3675
@@
 $EndComp
 $Comp
-L Diode:BAV99 D26
+L LoTI_Board-rescue:BAV99-Diode D26
 U 1 1 5E7ED96E
 P 9350 5075
@@
 $EndComp
 $Comp
-L Diode:BAV99 D26
+L LoTI_Board-rescue:BAV99-Diode D26
 U 2 1 5E7ED975
 P 9300 3275
@@
 	8625 3675 8850 3675
 $Comp
-L device:R R138
+L LoTI_Board-rescue:R-device R138
 U 1 1 5E7ED97F
 P 9000 3875
@@
 $EndComp
 $Comp
-L device:R R139
+L LoTI_Board-rescue:R-device R139
 U 1 1 5E7ED986
 P 9000 4075
@@
 	8625 4275 8850 4275
 $Comp
-L device:R R140
+L LoTI_Board-rescue:R-device R140
 U 1 1 5E7ED99D
 P 9000 4275
@@
 	8625 4475 8850 4475
 $Comp
-L device:R R141
+L LoTI_Board-rescue:R-device R141
 U 1 1 5E7ED9A8
 P 9000 4475
@@
 	8625 4675 8850 4675
 $Comp
-L device:R R142
+L LoTI_Board-rescue:R-device R142
 U 1 1 5E7ED9B3
 P 9000 4675
@@
 	9150 4675 10300 4675
 $Comp
-L Diode:BAV99 D29
+L LoTI_Board-rescue:BAV99-Diode D29
 U 1 1 5E7ED9BD
 P 9950 5075
@@
 $EndComp
 $Comp
-L Diode:BAV99 D30
+L LoTI_Board-rescue:BAV99-Diode D30
 U 1 1 5E7ED9C4
 P 10150 5075
@@
 $EndComp
 $Comp
-L Diode:BAV99 D31
+L LoTI_Board-rescue:BAV99-Diode D31
 U 1 1 5E7ED9CB
 P 10350 5075
@@
 	9750 4075 11375 4075
 $Comp
-L Diode:BAV99 D29
+L LoTI_Board-rescue:BAV99-Diode D29
 U 2 1 5E7ED9EE
 P 9900 3275
@@
 $EndComp
 $Comp
-L Diode:BAV99 D30
+L LoTI_Board-rescue:BAV99-Diode D30
 U 2 1 5E7ED9F5
 P 10100 3275
@@
 $EndComp
 $Comp
-L Diode:BAV99 D31
+L LoTI_Board-rescue:BAV99-Diode D31
 U 2 1 5E7ED9FC
 P 10300 3275
