File: kicad_hiltop_loti_board/HighSideOutputs.sch (KiCad schematic (older format))
At the start: 72 parts, among them Q10 ZXMN6A07F, Q11 ZXMN6A07F, Q12 ZXMN6A07F, Q13 ZXMN6A07F, Q14 ZXMN6A07F, Q7 ZXMN6A07F, Q8 ZXMN6A07F, Q9 ZXMN6A07F, U14 BTS4140N, U15 BTS4140N, U16 BTS4140N, U17 BTS4140N, U18 BTS4140N, U19 BTS4140N, U20 BTS4140N, U21 BTS4140N

Commit message: Rev A
Parts:
- C57, C58, C59, C60, C61, C62, C63, C64, C65, C66, C67, C68, C69, C70, C71, C72: symbol device:C -> LoTI_Board-rescue:C-device
- L10, L3, L4, L5, L6, L7, L8, L9: symbol device:Ferrite_Bead -> LoTI_Board-rescue:Ferrite_Bead-device
- Q10, Q11, Q12, Q13, Q14, Q7, Q8, Q9: symbol device:Q_NMOS_GSD -> LoTI_Board-rescue:Q_NMOS_GSD-device
- R100, R101, R102, R103, R104, R105, R106, R107, R108, R109, R110, R111, R112, R113, R114, R115, R116, R85, R86, R87, R88, R89, R90, R91, R92, R93, R94, R95, R96, R97, R98, R99: symbol device:R -> LoTI_Board-rescue:R-device
Changed lines of the file:
@@
 EESchema Schematic File Version 4
 LIBS:LoTI_Board-cache
-EELAYER 26 0
+EELAYER 29 0
 EELAYER END
 $Descr A3 16535 11693
@@
 $EndComp
 $Comp
-L device:Q_NMOS_GSD Q?
+L LoTI_Board-rescue:Q_NMOS_GSD-device Q?
 U 1 1 5CB48752
 P 3425 3400
@@
 $EndComp
 $Comp
-L device:R R?
+L LoTI_Board-rescue:R-device R?
 U 1 1 5CB48759
 P 2775 3400
@@
 $EndComp
 $Comp
-L device:R R?
+L LoTI_Board-rescue:R-device R?
 U 1 1 5CB48760
 P 3125 3675
@@
 	3525 3100 3525 3200
 $Comp
-L device:R R85
+L LoTI_Board-rescue:R-device R85
 U 1 1 5CB48C61
 P 2675 1750
@@
 $EndComp
 $Comp
-L device:R R91
+L LoTI_Board-rescue:R-device R91
 U 1 1 5CB48D37
 P 2950 1750
@@
 	2950 1425 2950 1600
 $Comp
-L device:Ferrite_Bead L3
+L LoTI_Board-rescue:Ferrite_Bead-device L3
 U 1 1 5CB4B291
 P 4350 2600
@@
 	3925 2600 4200 2600
 $Comp
-L device:C C60
+L LoTI_Board-rescue:C-device C60
 U 1 1 5CB4B566
 P 4775 2850
@@
 HS_CH1
 $Comp
-L device:C C57
+L LoTI_Board-rescue:C-device C57
 U 1 1 5CB4BB36
 P 2675 2450
@@
 $EndComp
 $Comp
-L device:Q_NMOS_GSD Q?
+L LoTI_Board-rescue:Q_NMOS_GSD-device Q?
 U 1 1 5CB527EB
 P 3425 6550
@@
 $EndComp
 $Comp
-L device:R R?
+L LoTI_Board-rescue:R-device R?
 U 1 1 5CB527F1
 P 2775 6550
@@
 $EndComp
 $Comp
-L device:R R?
+L LoTI_Board-rescue:R-device R?
 U 1 1 5CB527F7
 P 3125 6825
@@
 	3525 6250 3525 6350
 $Comp
-L device:R R86
+L LoTI_Board-rescue:R-device R86
 U 1 1 5CB52818
 P 2675 4900
@@
 $EndComp
 $Comp
-L device:R R92
+L LoTI_Board-rescue:R-device R92
 U 1 1 5CB5281E
 P 2950 4900
@@
 	2950 4575 2950 4750
 $Comp
-L device:Ferrite_Bead L4
+L LoTI_Board-rescue:Ferrite_Bead-device L4
 U 1 1 5CB52838
 P 4350 5750
@@
 	3925 5750 4200 5750
 $Comp
-L device:C C61
+L LoTI_Board-rescue:C-device C61
 U 1 1 5CB5283F
 P 4775 6000
@@
 HS_CH2
 $Comp
-L device:C C58
+L LoTI_Board-rescue:C-device C58
 U 1 1 5CB5284E
 P 2675 5600
@@
 $EndComp
 $Comp
-L device:Q_NMOS_GSD Q?
+L LoTI_Board-rescue:Q_NMOS_GSD-device Q?
 U 1 1 5CB54008
 P 3425 9750
@@
 $EndComp
 $Comp
-L device:R R?
+L LoTI_Board-rescue:R-device R?
 U 1 1 5CB5400E
 P 2775 9750
@@
 $EndComp
 $Comp
-L device:R R?
+L LoTI_Board-rescue:R-device R?
 U 1 1 5CB54014
 P 3125 10025
@@
 	3525 9450 3525 9550
 $Comp
-L device:R R87
+L LoTI_Board-rescue:R-device R87
 U 1 1 5CB54035
 P 2675 8100
@@
 $EndComp
 $Comp
-L device:R R93
+L LoTI_Board-rescue:R-device R93
 U 1 1 5CB5403B
 P 2950 8100
@@
 	2950 7775 2950 7950
 $Comp
-L device:Ferrite_Bead L5
+L LoTI_Board-rescue:Ferrite_Bead-device L5
 U 1 1 5CB54055
 P 4350 8950
@@
 	3925 8950 4200 8950
 $Comp
-L device:C C62
+L LoTI_Board-rescue:C-device C62
 U 1 1 5CB5405C
 P 4775 9200
@@
 HS_CH3
 $Comp
-L device:C C59
+L LoTI_Board-rescue:C-device C59
 U 1 1 5CB5406B
 P 2675 8800
@@
 $EndComp
 $Comp
-L device:Q_NMOS_GSD Q?
+L LoTI_Board-rescue:Q_NMOS_GSD-device Q?
 U 1 1 5CB58C92
 P 8475 3400
@@
 $EndComp
 $Comp
-L device:R R?
+L LoTI_Board-rescue:R-device R?
 U 1 1 5CB58C98
 P 7825 3400
@@
 $EndComp
 $Comp
-L device:R R?
+L LoTI_Board-rescue:R-device R?
 U 1 1 5CB58C9E
 P 8175 3675
@@
 	8575 3100 8575 3200
 $Comp
-L device:R R97
+L LoTI_Board-rescue:R-device R97
 U 1 1 5CB58CBF
 P 7725 1750
@@
 $EndComp
 $Comp
-L device:R R103
+L LoTI_Board-rescue:R-device R103
 U 1 1 5CB58CC5
 P 8000 1750
@@
 	8000 1425 8000 1600
 $Comp
-L device:Ferrite_Bead L6
+L LoTI_Board-rescue:Ferrite_Bead-device L6
 U 1 1 5CB58CDF
 P 9400 2600
@@
 	8975 2600 9250 2600
 $Comp
-L device:C C66
+L LoTI_Board-rescue:C-device C66
 U 1 1 5CB58CE6
 P 9825 2850
@@
 HS_CH4
 $Comp
-L device:C C63
+L LoTI_Board-rescue:C-device C63
 U 1 1 5CB58CF5
 P 7725 2450
@@
 $EndComp
 $Comp
-L device:Q_NMOS_GSD Q?
+L LoTI_Board-rescue:Q_NMOS_GSD-device Q?
 U 1 1 5CB58D11
 P 8475 6550
@@
 $EndComp
 $Comp
-L device:R R?
+L LoTI_Board-rescue:R-device R?
 U 1 1 5CB58D17
 P 7825 6550
@@
 $EndComp
 $Comp
-L device:R R?
+L LoTI_Board-rescue:R-device R?
 U 1 1 5CB58D1D
 P 8175 6825
@@
 	8575 6250 8575 6350
 $Comp
-L device:R R98
+L LoTI_Board-rescue:R-device R98
 U 1 1 5CB58D3E
 P 7725 4900
@@
 $EndComp
 $Comp
-L device:R R104
+L LoTI_Board-rescue:R-device R104
 U 1 1 5CB58D44
 P 8000 4900
@@
 	8000 4575 8000 4750
 $Comp
-L device:Ferrite_Bead L7
+L LoTI_Board-rescue:Ferrite_Bead-device L7
 U 1 1 5CB58D5E
 P 9400 5750
@@
 	8975 5750 9250 5750
 $Comp
-L device:C C67
+L LoTI_Board-rescue:C-device C67
 U 1 1 5CB58D65
 P 9825 6000
@@
 HS_CH5
 $Comp
-L device:C C64
+L LoTI_Board-rescue:C-device C64
 U 1 1 5CB58D74
 P 7725 5600
@@
 $EndComp
 $Comp
-L device:Q_NMOS_GSD Q?
+L LoTI_Board-rescue:Q_NMOS_GSD-device Q?
 U 1 1 5CB58D90
 P 8475 9750
@@
 $EndComp
 $Comp
-L device:R R?
+L LoTI_Board-rescue:R-device R?
 U 1 1 5CB58D96
 P 7825 9750
@@
 $EndComp
 $Comp
-L device:R R?
+L LoTI_Board-rescue:R-device R?
 U 1 1 5CB58D9C
 P 8175 10025
@@
 	8575 9450 8575 9550
 $Comp
-L device:R R99
+L LoTI_Board-rescue:R-device R99
 U 1 1 5CB58DBD
 P 7725 8100
@@
 $EndComp
 $Comp
-L device:R R105
+L LoTI_Board-rescue:R-device R105
 U 1 1 5CB58DC3
 P 8000 8100
@@
 	8000 7775 8000 7950
 $Comp
-L device:Ferrite_Bead L8
+L LoTI_Board-rescue:Ferrite_Bead-device L8
 U 1 1 5CB58DDD
 P 9400 8950
@@
 	8975 8950 9250 8950
 $Comp
-L device:C C68
+L LoTI_Board-rescue:C-device C68
 U 1 1 5CB58DE4
 P 9825 9200
@@
 HS_CH6
 $Comp
-L device:C C65
+L LoTI_Board-rescue:C-device C65
 U 1 1 5CB58DF3
 P 7725 8800
@@
 $EndComp
 $Comp
-L device:Q_NMOS_GSD Q?
+L LoTI_Board-rescue:Q_NMOS_GSD-device Q?
 U 1 1 5CB60C84
 P 13225 3400
@@
 $EndComp
 $Comp
-L device:R R?
+L LoTI_Board-rescue:R-device R?
 U 1 1 5CB60C8A
 P 12575 3400
@@
 $EndComp
 $Comp
-L device:R R?
+L LoTI_Board-rescue:R-device R?
 U 1 1 5CB60C90
 P 12925 3675
@@
 	13325 3100 13325 3200
 $Comp
-L device:R R109
+L LoTI_Board-rescue:R-device R109
 U 1 1 5CB60CB1
 P 12475 1750
@@
 $EndComp
 $Comp
-L device:R R113
+L LoTI_Board-rescue:R-device R113
 U 1 1 5CB60CB7
 P 12750 1750
@@
 	12750 1425 12750 1600
 $Comp
-L device:Ferrite_Bead L9
+L LoTI_Board-rescue:Ferrite_Bead-device L9
 U 1 1 5CB60CD1
 P 14150 2600
@@
 	13725 2600 14000 2600
 $Comp
-L device:C C71
+L LoTI_Board-rescue:C-device C71
 U 1 1 5CB60CD8
 P 14575 2850
@@
 HS_CH7
 $Comp
-L device:C C69
+L LoTI_Board-rescue:C-device C69
 U 1 1 5CB60CE7
 P 12475 2450
@@
 $EndComp
 $Comp
-L device:Q_NMOS_GSD Q?
+L LoTI_Board-rescue:Q_NMOS_GSD-device Q?
 U 1 1 5CB60D03
 P 13225 6550
@@
 $EndComp
 $Comp
-L device:R R?
+L LoTI_Board-rescue:R-device R?
 U 1 1 5CB60D09
 P 12575 6550
@@
 $EndComp
 $Comp
-L device:R R?
+L LoTI_Board-rescue:R-device R?
 U 1 1 5CB60D0F
 P 12925 6825
@@
 	13325 6250 13325 6350
 $Comp
-L device:R R110
+L LoTI_Board-rescue:R-device R110
 U 1 1 5CB60D30
 P 12475 4900
@@
 $EndComp
 $Comp
-L device:R R114
+L LoTI_Board-rescue:R-device R114
 U 1 1 5CB60D36
 P 12750 4900
@@
 	12750 4575 12750 4750
 $Comp
-L device:Ferrite_Bead L10
+L LoTI_Board-rescue:Ferrite_Bead-device L10
 U 1 1 5CB60D50
 P 14150 5750
@@
 	13725 5750 14000 5750
 $Comp
-L device:C C72
+L LoTI_Board-rescue:C-device C72
 U 1 1 5CB60D57
 P 14575 6000
@@
 HS_CH8
 $Comp
-L device:C C70
+L LoTI_Board-rescue:C-device C70
 U 1 1 5CB60D66
 P 12475 5600
