File: kicad_hiltop_loti_board/LoTI_Board.kicad_pcb (KiCad board)
At the start: 4 copper layers, 159.9 x 99.9 mm, 449 parts, among them J1 Conn_02x10_Odd_Even, J2 DB44_MALE_MountingHoles, J3 Conn_03x32_DIN41612, J4 RJ45-TRANS_VALCON, J5 USB_A, J6 Conn_02x08_Odd_Even, K1 HRS1KH-S, K2 HRS1KH-S, K3 HRS1KH-S, K4 HRS1KH-S, K5 HRS1KH-S, Q10 ZXMN6A07F, Q11 ZXMN6A07F, Q12 ZXMN6A07F, Q13 ZXMN6A07F, Q14 ZXMN6A07F, Q2 ZXMN6A07F, Q3 ZXMN6A07F, Q4 ZXMN6A07F, Q5 ZXMN6A07F, Q6 ZXMN6A07F, Q7 ZXMN6A07F, Q8 ZXMN6A07F, Q9 ZXMN6A07F, SW1 SW_Push, U1 INA250A4, U10 LAN9513, U11 MIC2026-1YM, U12 SP3003-02XJ, U13 CP2102N-A01-GQFN24, U14 BTS4140N, U15 BTS4140N, U16 BTS4140N, U17 BTS4140N, U18 BTS4140N, U19 BTS4140N, U2 LD1117S33TR_SOT223, U20 BTS4140N, U21 BTS4140N, U22 STM32F072RBTx, U3 AT25DN512CSSHF-B, U4 OPA197IDR, U5 OPA197IDR, U6 OPA197IDR, U7 OPA197IDR, U8 OPA197IDR, U9 93LCxxA, Y1 25MHz Crystal, Y2 8MHZ, Y3 ABS25-32.768KHZ-6-T

Commit message: updated drawing templates
Other:
- board text added: "Licensed under CERN OHL v1.2"
Changed lines of the file:
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@@
   (general
     (thickness 1.6)
-    (drawings 15)
+    (drawings 16)
     (tracks 3619)
     (zones 0)
@@
   )
   (page A4)
+  (title_block
+    (title "LoTI Board")
+    (date 2019-07-03)
+    (rev A)
+    (company "Devtank Ltd")
+  )
   (layers
     (0 F.Cu signal)
@@
     )
   )
+  (gr_text "Licensed under \nCERN OHL v1.2" (at 71.3 68.975) (layer F.SilkS)
+    (effects (font (size 1 1) (thickness 0.2)) (justify left))
+  )
   (gr_line (start 214.925 45.075) (end 214.925 45.075) (angle 90) (layer Edge.Cuts) (width 0.15))
   (gr_text S/N: (at 72.644 51.054 180) (layer B.SilkS)
@@
   (via (at 78.725 86.225) (size 1) (drill 0.5) (layers F.Cu B.Cu) (net 1))
   (via (at 76.85 71.475) (size 1) (drill 0.5) (layers F.Cu B.Cu) (net 1))
-  (via (at 82.35 69.025) (size 1) (drill 0.5) (layers F.Cu B.Cu) (net 1))
+  (via (at 83.475 68.55) (size 1) (drill 0.5) (layers F.Cu B.Cu) (net 1))
   (via (at 85.4 65.725) (size 1) (drill 0.5) (layers F.Cu B.Cu) (net 1))
   (via (at 77.025 67.05) (size 1) (drill 0.5) (layers F.Cu B.Cu) (net 1))

Commit message: Rev B updates
Parts:
- added C54: 100nF, Capacitor_SMD:C_0603_1608Metric, F.Cu at (130.2, 55.5)
- added R152: 47K, Resistor_SMD:R_0603_1608Metric, F.Cu at (156.7, 60.4)
- added U23: M74VHC1GT14DFT2G, Package_TO_SOT_SMD:SOT-353_SC-70-5, F.Cu at (133.9, 54.1)
- C38: value 0.1uF -> 100nF
- D10, D13, D2, D3, D6, D7: value LED -> GRN
- D12: value GRN -> RED
- D32: value 1N4002 -> MBR230LSFT1G
- L10, L11, L3, L4, L5, L6, L7, L8, L9: value Ferrite_Bead -> 2A/0.05DCR
- R117: value 10K -> DNF
- R78: value 0R -> 24K
- R79, R80: value 330R -> 0R
- R8, R9: value 0R -> DNF
- U4, U5, U6, U7, U8: value OPA197IDR -> AD8646
- moved TP33 1.20 mm to (130.4, 53.8)
- moved TP34 0.77 mm to (133.1, 56.5)
- turned D10 to 270 degrees
- turned D2 to 270 degrees
- turned D3 to 270 degrees
- turned D6 to 270 degrees
- turned D7 to 270 degrees
Connections:
- D10 pad 1: +5V -> Net-(D10-Pad1)
- D10 pad 2: Net-(D10-Pad2) -> +5V
- D2 pad 1: +5V -> Net-(D2-Pad1)
- D2 pad 2: Net-(D2-Pad2) -> +5V
- D3 pad 1: +5V -> Net-(D3-Pad1)
- D3 pad 2: Net-(D3-Pad2) -> +5V
- D6 pad 1: +5V -> Net-(D6-Pad1)
- D6 pad 2: Net-(D6-Pad2) -> +5V
- D7 pad 1: +5V -> Net-(D7-Pad1)
- D7 pad 2: Net-(D7-Pad2) -> +5V
- J2 pad 20: (no net) -> Net-(J2-Pad20)
- J3 pad 11a: (no net) -> /FPGA_IO1
- J3 pad 11b: (no net) -> /SPI0_CS0
- J3 pad 12a: (no net) -> /FPGA_IO2
- J3 pad 12b: (no net) -> /SPI0_CS1
- J3 pad 12c: (no net) -> /I2C0_SDA
- J3 pad 13a: (no net) -> /FPGA_IO3
- J3 pad 13c: (no net) -> /I2C0_SCL
- J3 pad 14a: (no net) -> /FPGA_IO4
- J3 pad 14b: (no net) -> /SPI1_MOSI
- J3 pad 15a: (no net) -> /FPGA_IO5
- J3 pad 15b: (no net) -> /SPI1_MISO
- J3 pad 15c: (no net) -> /I2C1_SDA
- J3 pad 16a: (no net) -> /FPGA_IO6
- J3 pad 16b: (no net) -> /SPI1_CLK
- J3 pad 16c: (no net) -> /I2C1_SCL
- J3 pad 17a: (no net) -> /FPGA_IO7
- J3 pad 17b: (no net) -> /SPI1_CS0
- J3 pad 18a: (no net) -> /FPGA_IO8
- J3 pad 18b: (no net) -> /SPI1_CS1
- J3 pad 18c: (no net) -> /MBRD_IO4
- J3 pad 19a: (no net) -> /FPGA_IO9
- J3 pad 19b: (no net) -> /SPI1_CS2
- J3 pad 19c: (no net) -> /MBRD_IO5
- J3 pad 20a: (no net) -> /FPGA_IO10
- J3 pad 20b: (no net) -> /GPIO1_MBRD
- J3 pad 20c: (no net) -> /MBRD_IO6
- J3 pad 21b: (no net) -> /GPIO2_MBRD
- J3 pad 21c: (no net) -> /MBRD_IO7
- J3 pad 22a: (no net) -> /MBRD_IO8
- J3 pad 22b: (no net) -> /GPIO3_MBRD
- J3 pad 22c: (no net) -> /PWM0
- J3 pad 23a: (no net) -> /MBRD_IO9
- J3 pad 23c: (no net) -> /PWM1
- J3 pad 24a: (no net) -> /MBRD_IO10
- J3 pad 24b: (no net) -> /SYS_CLK
- J3 pad 25a: (no net) -> /LCOM_1
- J3 pad 25b: (no net) -> /SYS_TRIG
- J3 pad 25c: (no net) -> /RCOM_1
- J3 pad 26a: (no net) -> /LCOM_2
- J3 pad 26c: (no net) -> /RCOM_2
- J3 pad 27a: (no net) -> /LCOM_3
- J3 pad 27b: (no net) -> /SHUTDOWN
- J3 pad 27c: (no net) -> /RCOM_3
- J3 pad 28a: (no net) -> /LCOM_4
- J3 pad 28c: (no net) -> /RCOM_4
- J3 pad 29a: (no net) -> /LCOM_5
- J3 pad 29c: (no net) -> /RCOM_5
- J3 pad 2a: (no net) -> /LVDSCLK+
- J3 pad 30a: (no net) -> /LCOM_6
- J3 pad 30c: (no net) -> /RCOM_6
- J3 pad 31a: (no net) -> /LCOM_7
- J3 pad 31c: (no net) -> /RCOM_7
- J3 pad 32a: (no net) -> /LCOM_8
- J3 pad 32c: (no net) -> /RCOM_8
- J3 pad 3a: (no net) -> /LVDSCLK-
- J3 pad 5a: (no net) -> /LVDS_MOSI+
- J3 pad 6a: (no net) -> /LVDS_MOSI-
- J3 pad 7b: (no net) -> GND
- J3 pad 7c: GND -> +3V3_BP
- J3 pad 8a: (no net) -> /LVDS_MISO+
- J3 pad 9a: (no net) -> /LVDS_MISO-
- R48 pad 2: Net-(D2-Pad2) -> Net-(D2-Pad1)
- R49 pad 2: Net-(D3-Pad2) -> Net-(D3-Pad1)
- R54 pad 2: Net-(D6-Pad2) -> Net-(D6-Pad1)
- R55 pad 2: Net-(D7-Pad2) -> Net-(D7-Pad1)
- R60 pad 2: Net-(D10-Pad2) -> Net-(D10-Pad1)
- R79 pad 1: /STM_BOOT0 -> Net-(R79-Pad1)
- U10 pad 13: (no net) -> Net-(U10-Pad13)
- U10 pad 18: (no net) -> Net-(U10-Pad18)
- U10 pad 24: (no net) -> /USB_Controller/EECS
- U10 pad 31: (no net) -> Net-(U10-Pad31)
- U10 pad 35: (no net) -> Net-(U10-Pad35)
- U10 pad 36: (no net) -> Net-(U10-Pad36)
- U10 pad 37: (no net) -> Net-(U10-Pad37)
- U10 pad 42: (no net) -> Net-(U10-Pad42)
- U10 pad 43: (no net) -> Net-(U10-Pad43)
- U10 pad 45: (no net) -> Net-(U10-Pad45)
- U10 pad 47: (no net) -> Net-(U10-Pad47)
- U10 pad 8: (no net) -> Net-(U10-Pad8)
- U10 pad 9: (no net) -> Net-(U10-Pad9)
- U11 pad 3: (no net) -> Net-(U11-Pad3)
- U11 pad 4: (no net) -> Net-(U11-Pad4)
- U11 pad 5: (no net) -> Net-(U11-Pad5)
- U12 pad 1: (no net) -> Net-(U12-Pad1)
- U13 pad 1: (no net) -> Net-(U13-Pad1)
- U13 pad 10: (no net) -> Net-(U13-Pad10)
- U13 pad 15: (no net) -> Net-(U13-Pad15)
- U13 pad 16: (no net) -> Net-(U13-Pad16)
- U13 pad 17: (no net) -> Net-(U13-Pad17)
- U13 pad 18: (no net) -> Net-(U13-Pad18)
- U13 pad 19: (no net) -> Net-(U13-Pad19)
- U13 pad 22: (no net) -> Net-(U13-Pad22)
- U13 pad 23: (no net) -> Net-(U13-Pad23)
- U13 pad 24: (no net) -> Net-(U13-Pad24)
- U22 pad 1: (no net) -> Net-(U22-Pad1)
- U9 pad 6: (no net) -> Net-(U9-Pad6)
- U9 pad 7: (no net) -> Net-(U9-Pad7)
- Y2 pad 2: (no net) -> Net-(Y2-Pad2)
- Y2 pad 4: (no net) -> Net-(Y2-Pad4)
- Y3 pad 2: (no net) -> Net-(Y3-Pad2)
- Y3 pad 3: (no net) -> Net-(Y3-Pad3)
Routing:
- net /STM_BOOT0: track 36.1 -> 30.7 mm
- net Net-(D7-Pad2): track 4.47 -> 0.00 mm
- net Net-(D7-Pad1): track 0.00 -> 4.47 mm
- net GND: track 222.2 -> 226.3 mm, vias 215 -> 217
- net Net-(R79-Pad1): track 0.00 -> 3.42 mm
- net Net-(D3-Pad2): track 3.09 -> 0.00 mm
- net Net-(D3-Pad1): track 0.00 -> 3.09 mm
- net Net-(D2-Pad2): track 3.06 -> 0.00 mm
- net Net-(D2-Pad1): track 0.00 -> 3.06 mm
- net Net-(D6-Pad2): track 2.80 -> 0.00 mm
- net Net-(D6-Pad1): track 0.00 -> 2.80 mm
- net Net-(D10-Pad2): track 2.77 -> 0.00 mm
- net Net-(D10-Pad1): track 0.00 -> 2.77 mm
- net +3V3_BP: track 21.8 -> 24.3 mm
- net +3V3: track 105.7 -> 108.1 mm, vias 53 -> 54
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Other:
- board size 159.9 x 99.9 mm -> 159.1 x 99.9 mm
- board text added: "(c) Copyright 2021 Devtank Ltd Licensed under CERN-OHL-W V2.0 https://cern-ohl.web.cern.ch/"
- board text added: "LoTI Board PN: 304-006 Rev: B"
- board text removed: "Licensed under CERN OHL v1.2"
- board text removed: "LoTI Board PN: 304-006 Rev: A"
