File: kicad_hiltop_loti_board/LoTI_Board.sch (KiCad schematic (older format))
At the start: 160 parts, among them J1 Conn_02x10_Odd_Even, J2 DB44_MALE_MountingHoles, J3 Conn_03x32_DIN41612, J4 RJ45-TRANS_VALCON, J5 USB_A, J6 Conn_02x08_Odd_Even, U1 INA250A4, U2 LD1117S33TR_SOT223, U3 AT25DN512CSSHF-B

Commit message: Rev B updates
Parts:
- D33: value BAT42W -> DNF
- J1: value Conn_02x10_Odd_Even -> AMPMODU HE14 20WAY
- J6: value Conn_02x08_Odd_Even -> AMPMODU HE14 16WAY
- R12, R148: value 0R -> DNF; Devtank 101-005 -> (none)
- R13: value 2.7K -> DNF
- R144, R146, R8, R9: value 0R -> DNF
- R145: value 1.25K -> DNF
Changed lines of the file:
@@
 EESchema Schematic File Version 4
-LIBS:LoTI_Board-cache
-EELAYER 29 0
+EELAYER 30 0
 EELAYER END
 $Descr A2 23386 16535
@@
 Sheet 1 8
 Title "LoTI Board"
-Date "2019-07-03"
-Rev "Rev A"
+Date "2020-07-01"
+Rev "Rev B"
 Comp "Devtank Ltd"
 Comment1 ""
@@
 	0    -1   -1   0
 $EndComp
-$Sheet
-S 14350 9700 1925 2800
-U 5C87E9AC
-F0 "USB_Controller" 60
-F1 "USB_Controller.sch" 60
-F2 "USB0_UP_P" B L 14350 12325 60
-F3 "USB0_UP_N" B L 14350 12200 60
-F4 "USB2_DN_P" B R 16275 12325 60
-F5 "USB2_DN_N" B R 16275 12200 60
-F6 "USB3_DN_P" B R 16275 12075 60
-F7 "USB3_DN_N" B R 16275 11950 60
-F8 "USB4_DN_P" B R 16275 11825 60
-F9 "USB4_DN_N" B R 16275 11700 60
-F10 "USB4_PWR" O R 16275 11500 60
-F11 "TXP" O R 16275 11275 60
-F12 "TXN" O R 16275 11150 60
-F13 "RXP" O R 16275 11025 60
-F14 "RXN" O R 16275 10900 60
-F15 "nFDX_LED" O R 16275 10050 60
-F16 "nLNKA_LED" O R 16275 9900 60
-F17 "nSPD_LED" O R 16275 10200 60
-F18 "RESET" I L 14350 11875 60
-$EndSheet
 Text Label 17275 12150 2    60   ~ 0
 nFDX_LED
@@
 P 18175 8100
 F 0 "R9" H 18075 8025 50  0000 C CNN
-F 1 "0R" H 18075 8125 50  0000 C CNN
+F 1 "DNF" H 18075 8125 50  0000 C CNN
 F 2 "Resistor_SMD:R_1206_3216Metric" V 18105 8100 50  0001 C CNN
 F 3 "" H 18175 8100 50  0001 C CNN
@@
 P 17925 8100
 F 0 "R8" H 17825 8025 50  0000 C CNN
-F 1 "0R" H 17825 8125 50  0000 C CNN
+F 1 "DNF" H 17825 8125 50  0000 C CNN
 F 2 "Resistor_SMD:R_1206_3216Metric" V 17855 8100 50  0001 C CNN
 F 3 "" H 17925 8100 50  0001 C CNN
@@
 P 2650 9175
 F 0 "J1" H 2700 9792 50  0000 C CNN
-F 1 "Conn_02x10_Odd_Even" H 2700 9701 50  0000 C CNN
+F 1 "AMPMODU HE14 20WAY" H 2700 9701 50  0000 C CNN
 F 2 "Connector_IDC:IDC-Header_2x10_P2.54mm_Vertical" H 2650 9175 50  0001 C CNN
 F 3 "~" H 2650 9175 50  0001 C CNN
@@
 P 22200 10800
 F 0 "D33" V 22246 10721 50  0000 R CNN
-F 1 "BAT42W" V 22155 10721 50  0000 R CNN
+F 1 "DNF" V 22155 10721 50  0000 R CNN
 F 2 "Diode_SMD:D_SOD-123" H 22200 10800 50  0001 C CNN
 F 3 "" H 22200 10800 50  0001 C CNN
@@
 P 22225 11350
 F 0 "R13" V 22175 11100 50  0000 C CNN
-F 1 "2.7K" V 22175 11550 50  0000 C CNN
+F 1 "DNF" V 22175 11550 50  0000 C CNN
 F 2 "Resistor_SMD:R_0603_1608Metric" V 22155 11350 50  0001 C CNN
 F 3 "" H 22225 11350 50  0001 C CNN
@@
 P 22225 11950
 F 0 "R145" V 22175 11700 50  0000 C CNN
-F 1 "1.25K" V 22175 12150 50  0000 C CNN
+F 1 "DNF" V 22175 12150 50  0000 C CNN
 F 2 "Resistor_SMD:R_0603_1608Metric" V 22155 11950 50  0001 C CNN
 F 3 "" H 22225 11950 50  0001 C CNN
@@
 P 22225 11800
 F 0 "R144" V 22175 11550 50  0000 C CNN
-F 1 "0R" V 22175 12000 50  0000 C CNN
+F 1 "DNF" V 22175 12000 50  0000 C CNN
 F 2 "Resistor_SMD:R_0603_1608Metric" V 22155 11800 50  0001 C CNN
 F 3 "" H 22225 11800 50  0001 C CNN
@@
 P 22225 12400
 F 0 "R146" V 22175 12150 50  0000 C CNN
-F 1 "0R" V 22175 12600 50  0000 C CNN
+F 1 "DNF" V 22175 12600 50  0000 C CNN
 F 2 "Resistor_SMD:R_0603_1608Metric" V 22155 12400 50  0001 C CNN
 F 3 "" H 22225 12400 50  0001 C CNN
@@
 P 22225 11200
 F 0 "R12" V 22175 10950 50  0000 C CNN
-F 1 "0R" V 22175 11400 50  0000 C CNN
+F 1 "DNF" V 22175 11400 50  0000 C CNN
 F 2 "Resistor_SMD:R_0603_1608Metric" V 22155 11200 50  0001 C CNN
 F 3 "" H 22225 11200 50  0001 C CNN
-F 4 "101-005" H 0   0   50  0001 C CNN "Devtank"
+F 4 "" H 0   0   50  0001 C CNN "Devtank"
 	1    22225 11200
 	0    1    1    0
@@
 P 22400 11025
 F 0 "R148" V 22350 10775 50  0000 C CNN
-F 1 "0R" V 22350 11225 50  0000 C CNN
+F 1 "DNF" V 22350 11225 50  0000 C CNN
 F 2 "Resistor_SMD:R_0603_1608Metric" V 22330 11025 50  0001 C CNN
 F 3 "" H 22400 11025 50  0001 C CNN
-F 4 "101-005" H 0   0   50  0001 C CNN "Devtank"
+F 4 "" H 0   0   50  0001 C CNN "Devtank"
 	1    22400 11025
 	0    1    1    0
@@
 P 5550 9175
 F 0 "J6" H 5600 9692 50  0000 C CNN
-F 1 "Conn_02x08_Odd_Even" H 5600 9601 50  0000 C CNN
+F 1 "AMPMODU HE14 16WAY" H 5600 9601 50  0000 C CNN
 F 2 "Connector_IDC:IDC-Header_2x08_P2.54mm_Vertical" H 5550 9175 50  0001 C CNN
 F 3 "~" H 5550 9175 50  0001 C CNN
@@
 Wire Wire Line
 	14775 9225 14875 9225
+$Sheet
+S 14350 9700 1925 2800
+U 5C87E9AC
+F0 "USB_Controller" 60
+F1 "USB_Controller.sch" 60
+F2 "USB0_UP_P" B L 14350 9875 60
+F3 "USB0_UP_N" B L 14350 10000 60
+F4 "USB2_DN_P" B R 16275 9875 60
+F5 "USB2_DN_N" B R 16275 10000 60
+F6 "USB3_DN_P" B R 16275 10125 60
+F7 "USB3_DN_N" B R 16275 10250 60
+F8 "USB4_DN_P" B R 16275 10375 60
+F9 "USB4_DN_N" B R 16275 10500 60
+F10 "USB4_PWR" O R 16275 10700 60
+F11 "TXP" O R 16275 10925 60
+F12 "TXN" O R 16275 11050 60
+F13 "RXP" O R 16275 11175 60
+F14 "RXN" O R 16275 11300 60
+F15 "nFDX_LED" O R 16275 12150 60
+F16 "nLNKA_LED" O R 16275 12300 60
+F17 "nSPD_LED" O R 16275 12000 60
+F18 "RESET" I L 14350 10325 60
+$EndSheet
 $EndSCHEMATC
