File: kicad_hiltop_loti_board/RelayOutputs.sch (KiCad schematic (older format))
At the start: 35 parts, among them K1 HRS1KH-S, K2 HRS1KH-S, K3 HRS1KH-S, K4 HRS1KH-S, K5 HRS1KH-S, Q2 ZXMN6A07F, Q3 ZXMN6A07F, Q4 ZXMN6A07F, Q5 ZXMN6A07F, Q6 ZXMN6A07F

Commit message: Rev A
Parts:
- D10, D2, D3, D6, D7: symbol device:LED -> LoTI_Board-rescue:LED-device
- D11, D4, D5, D8, D9: symbol device:D_Schottky -> LoTI_Board-rescue:D_Schottky-device
- K1, K2, K3, K4, K5: symbol Relay:G5Q-1 -> LoTI_Board-rescue:G5Q-1-Relay
- Q2, Q3, Q4, Q5, Q6: symbol device:Q_NMOS_GSD -> LoTI_Board-rescue:Q_NMOS_GSD-device
- R48, R49, R50, R51, R52, R53, R54, R55, R56, R57, R58, R59, R60, R61, R62: symbol device:R -> LoTI_Board-rescue:R-device
Changed lines of the file:
@@
 EESchema Schematic File Version 4
 LIBS:LoTI_Board-cache
-EELAYER 26 0
+EELAYER 29 0
 EELAYER END
 $Descr A3 16535 11693
@@
 $EndDescr
 $Comp
-L Relay:G5Q-1 K?
+L LoTI_Board-rescue:G5Q-1-Relay K?
 U 1 1 5BE5E5DE
 P 4200 2950
@@
 $EndComp
 $Comp
-L device:D_Schottky D?
+L LoTI_Board-rescue:D_Schottky-device D?
 U 1 1 5BE5E5E5
 P 3500 2800
@@
 $EndComp
 $Comp
-L device:Q_NMOS_GSD Q?
+L LoTI_Board-rescue:Q_NMOS_GSD-device Q?
 U 1 1 5BE5E5EC
 P 4100 3525
@@
 $EndComp
 $Comp
-L device:R R?
+L LoTI_Board-rescue:R-device R?
 U 1 1 5BE5E5F3
 P 3450 3525
@@
 $EndComp
 $Comp
-L device:R R?
+L LoTI_Board-rescue:R-device R?
 U 1 1 5BE5E5FA
 P 3800 3800
@@
 	4600 3225 5400 3225
 $Comp
-L device:LED D?
+L LoTI_Board-rescue:LED-device D?
 U 1 1 5BE5E626
 P 3025 2575
@@
 $EndComp
 $Comp
-L device:R R?
+L LoTI_Board-rescue:R-device R?
 U 1 1 5BE5E62D
 P 3025 2975
@@
 	4200 3250 4200 3325
 $Comp
-L Relay:G5Q-1 K?
+L LoTI_Board-rescue:G5Q-1-Relay K?
 U 1 1 5BE5FACF
 P 4200 5575
@@
 $EndComp
 $Comp
-L device:D_Schottky D?
+L LoTI_Board-rescue:D_Schottky-device D?
 U 1 1 5BE5FAD5
 P 3500 5425
@@
 $EndComp
 $Comp
-L device:Q_NMOS_GSD Q?
+L LoTI_Board-rescue:Q_NMOS_GSD-device Q?
 U 1 1 5BE5FADB
 P 4100 6150
@@
 $EndComp
 $Comp
-L device:R R?
+L LoTI_Board-rescue:R-device R?
 U 1 1 5BE5FAE1
 P 3450 6150
@@
 $EndComp
 $Comp
-L device:R R?
+L LoTI_Board-rescue:R-device R?
 U 1 1 5BE5FAE7
 P 3800 6425
@@
 	4600 5850 5400 5850
 $Comp
-L device:LED D?
+L LoTI_Board-rescue:LED-device D?
 U 1 1 5BE5FB12
 P 3025 5200
@@
 $EndComp
 $Comp
-L device:R R?
+L LoTI_Board-rescue:R-device R?
 U 1 1 5BE5FB18
 P 3025 5600
@@
 	4200 5875 4200 5950
 $Comp
-L Relay:G5Q-1 K?
+L LoTI_Board-rescue:G5Q-1-Relay K?
 U 1 1 5BE624A2
 P 8325 2950
@@
 $EndComp
 $Comp
-L device:D_Schottky D?
+L LoTI_Board-rescue:D_Schottky-device D?
 U 1 1 5BE624A8
 P 7625 2800
@@
 $EndComp
 $Comp
-L device:Q_NMOS_GSD Q?
+L LoTI_Board-rescue:Q_NMOS_GSD-device Q?
 U 1 1 5BE624AE
 P 8225 3525
@@
 $EndComp
 $Comp
-L device:R R?
+L LoTI_Board-rescue:R-device R?
 U 1 1 5BE624B4
 P 7575 3525
@@
 $EndComp
 $Comp
-L device:R R?
+L LoTI_Board-rescue:R-device R?
 U 1 1 5BE624BA
 P 7925 3800
@@
 	8725 3225 9525 3225
 $Comp
-L device:LED D?
+L LoTI_Board-rescue:LED-device D?
 U 1 1 5BE624E5
 P 7150 2575
@@
 $EndComp
 $Comp
-L device:R R?
+L LoTI_Board-rescue:R-device R?
 U 1 1 5BE624EB
 P 7150 2975
@@
 	8325 3250 8325 3325
 $Comp
-L Relay:G5Q-1 K?
+L LoTI_Board-rescue:G5Q-1-Relay K?
 U 1 1 5BE62503
 P 8325 5575
@@
 $EndComp
 $Comp
-L device:D_Schottky D?
+L LoTI_Board-rescue:D_Schottky-device D?
 U 1 1 5BE62509
 P 7625 5425
@@
 $EndComp
 $Comp
-L device:Q_NMOS_GSD Q?
+L LoTI_Board-rescue:Q_NMOS_GSD-device Q?
 U 1 1 5BE6250F
 P 8225 6150
@@
 $EndComp
 $Comp
-L device:R R?
+L LoTI_Board-rescue:R-device R?
 U 1 1 5BE62515
 P 7575 6150
@@
 $EndComp
 $Comp
-L device:R R?
+L LoTI_Board-rescue:R-device R?
 U 1 1 5BE6251B
 P 7925 6425
@@
 	8725 5850 9525 5850
 $Comp
-L device:LED D?
+L LoTI_Board-rescue:LED-device D?
 U 1 1 5BE62546
 P 7150 5200
@@
 $EndComp
 $Comp
-L device:R R?
+L LoTI_Board-rescue:R-device R?
 U 1 1 5BE6254C
 P 7150 5600
@@
 OUT4_COM
 $Comp
-L Relay:G5Q-1 K?
+L LoTI_Board-rescue:G5Q-1-Relay K?
 U 1 1 5C37B22A
 P 12600 2950
@@
 $EndComp
 $Comp
-L device:D_Schottky D?
+L LoTI_Board-rescue:D_Schottky-device D?
 U 1 1 5C37B230
 P 11900 2800
@@
 $EndComp
 $Comp
-L device:Q_NMOS_GSD Q?
+L LoTI_Board-rescue:Q_NMOS_GSD-device Q?
 U 1 1 5C37B236
 P 12500 3525
@@
 $EndComp
 $Comp
-L device:R R?
+L LoTI_Board-rescue:R-device R?
 U 1 1 5C37B23C
 P 11850 3525
@@
 $EndComp
 $Comp
-L device:R R?
+L LoTI_Board-rescue:R-device R?
 U 1 1 5C37B242
 P 12200 3800
@@
 	13000 3225 13800 3225
 $Comp
-L device:LED D?
+L LoTI_Board-rescue:LED-device D?
 U 1 1 5C37B26D
 P 11425 2575
@@
 $EndComp
 $Comp
-L device:R R?
+L LoTI_Board-rescue:R-device R?
 U 1 1 5C37B273
 P 11425 2975

Commit message: Rev B updates
Connections:
- net +5V: now also D10.2 (A), D2.2 (A), D3.2 (A), D6.2 (A), D7.2 (A); no longer D10.1 (K), D2.1 (K), D3.1 (K), D6.1 (K), D7.1 (K)
- net at R48.2: now also D2.1 (K); no longer D2.2 (A)
- net at R49.2: now also D3.1 (K); no longer D3.2 (A)
- net at R54.2: now also D6.1 (K); no longer D6.2 (A)
- net at R55.2: now also D7.1 (K); no longer D7.2 (A)
- net at R60.2: now also D10.1 (K); no longer D10.2 (A)
Other:
- moved on the sheet: D10, D2, D3, D6, D7
Changed lines of the file:
@@
 EESchema Schematic File Version 4
-LIBS:LoTI_Board-cache
-EELAYER 29 0
+EELAYER 30 0
 EELAYER END
 $Descr A3 16535 11693
@@
 Sheet 3 8
 Title "LoTI Board"
-Date "2019-07-03"
-Rev "Rev A"
+Date "2020-07-01"
+Rev "Rev B"
 Comp "Devtank Ltd"
 Comment1 ""
@@
 F 4 "110-002" H 0   0   50  0001 C CNN "Devtank"
 	1    3025 2575
-	0    1    1    0
+	0    -1   -1   0
 $EndComp
 $Comp
@@
 F 4 "110-002" H 0   0   50  0001 C CNN "Devtank"
 	1    3025 5200
-	0    1    1    0
+	0    -1   -1   0
 $EndComp
 $Comp
@@
 F 4 "110-002" H 0   0   50  0001 C CNN "Devtank"
 	1    7150 2575
-	0    1    1    0
+	0    -1   -1   0
 $EndComp
 $Comp
@@
 F 4 "110-002" H 0   0   50  0001 C CNN "Devtank"
 	1    7150 5200
-	0    1    1    0
+	0    -1   -1   0
 $EndComp
 $Comp
@@
 F 4 "110-002" H 0   0   50  0001 C CNN "Devtank"
 	1    11425 2575
-	0    1    1    0
-$EndComp
-$Comp
+	0    -1   -1   0
+$EndComp
+$Comp
