File: kicad_hiltop_loti_board/STM_Micro.sch (KiCad schematic (older format))
At the start: 25 parts, among them SW1 SW_Push, U22 STM32F072RBTx, Y2 8MHZ, Y3 ABS25-32.768KHZ-6-T

Commit message: Rev A
Parts:
- C73, C74, C75, C76, C77, C78, C79, C80, C81, C82: symbol device:C -> LoTI_Board-rescue:C-device
- D13: symbol device:LED -> LoTI_Board-rescue:LED-device
- L11: symbol device:Ferrite_Bead -> LoTI_Board-rescue:Ferrite_Bead-device
- R117, R118, R119, R120, R121, R122, R123, R124: symbol device:R -> LoTI_Board-rescue:R-device
- TP126: symbol Connector:Test_Point -> LoTI_Board-rescue:Test_Point-Connector
- U22: symbol MCU_ST_STM32:STM32F072RBTx -> LoTI_Board-rescue:STM32F072RBTx-MCU_ST_STM32
- Y2: symbol device:Crystal_GND24 -> LoTI_Board-rescue:Crystal_GND24-device
- Y3: symbol device:Crystal_GND23 -> LoTI_Board-rescue:Crystal_GND23-device
Changed lines of the file:
@@
 EESchema Schematic File Version 4
 LIBS:LoTI_Board-cache
-EELAYER 26 0
+EELAYER 29 0
 EELAYER END
 $Descr A3 16535 11693
@@
 $EndDescr
 $Comp
-L MCU_ST_STM32:STM32F072RBTx U22
+L LoTI_Board-rescue:STM32F072RBTx-MCU_ST_STM32 U22
 U 1 1 5F956EB6
 P 7400 4675
@@
 $EndComp
 $Comp
-L device:Ferrite_Bead L11
+L LoTI_Board-rescue:Ferrite_Bead-device L11
 U 1 1 5F957109
 P 8225 2025
@@
 	8525 2025 8375 2025
 $Comp
-L device:C C82
+L LoTI_Board-rescue:C-device C82
 U 1 1 5F957430
 P 7875 2250
@@
 $EndComp
 $Comp
-L device:C C73
+L LoTI_Board-rescue:C-device C73
 U 1 1 5F957A1A
 P 2125 1625
@@
 $EndComp
 $Comp
-L device:C C74
+L LoTI_Board-rescue:C-device C74
 U 1 1 5F957BC6
 P 2575 1625
@@
 $EndComp
 $Comp
-L device:C C79
+L LoTI_Board-rescue:C-device C79
 U 1 1 5F957C44
 P 3025 1625
@@
 $EndComp
 $Comp
-L device:C C80
+L LoTI_Board-rescue:C-device C80
 U 1 1 5F957C84
 P 3475 1625
@@
 	4400 3075 3825 3075
 $Comp
-L device:R R120
+L LoTI_Board-rescue:R-device R120
 U 1 1 5F95CC59
 P 2725 2850
@@
 $EndComp
 $Comp
-L device:R R117
+L LoTI_Board-rescue:R-device R117
 U 1 1 5F95CDB1
 P 2550 3500
@@
 BOOT0
 $Comp
-L device:C C81
+L LoTI_Board-rescue:C-device C81
 U 1 1 5F9616D2
 P 3825 3550
@@
 $EndComp
 $Comp
-L device:Crystal_GND23 Y3
+L LoTI_Board-rescue:Crystal_GND23-device Y3
 U 1 1 5F964614
 P 3225 6550
@@
 	3575 6525 4100 6525
 $Comp
-L device:C C77
+L LoTI_Board-rescue:C-device C77
 U 1 1 5F96D367
 P 2850 6275
@@
 Connection ~ 3225 6275
 $Comp
-L device:C C78
+L LoTI_Board-rescue:C-device C78
 U 1 1 5F96FC00
 P 2850 6825
@@
 Connection ~ 3225 6825
 $Comp
-L device:Crystal_GND24 Y2
+L LoTI_Board-rescue:Crystal_GND24-device Y2
 U 1 1 5F97410A
 P 3050 4325
@@
 	3050 4075 3050 4175
 $Comp
-L device:C C75
+L LoTI_Board-rescue:C-device C75
 U 1 1 5F97DA85
 P 2825 4075
@@
 	2550 4075 2675 4075
 $Comp
-L device:C C76
+L LoTI_Board-rescue:C-device C76
 U 1 1 5F97DA93
 P 2825 4625
@@
 	10400 3275 11800 3275
 $Comp
-L device:R R122
+L LoTI_Board-rescue:R-device R122
 U 1 1 5FA3B65A
 P 11325 3075
@@
 	11475 3075 11800 3075
 $Comp
-L device:R R123
+L LoTI_Board-rescue:R-device R123
 U 1 1 5FA3B8E4
 P 11325 3175
@@
 	11475 3175 11800 3175
 $Comp
-L device:R R118
+L LoTI_Board-rescue:R-device R118
 U 1 1 5FA60497
 P 2675 5775
@@
 	2525 5775 2200 5775
 $Comp
-L device:R R119
+L LoTI_Board-rescue:R-device R119
 U 1 1 5FA6049E
 P 2675 5875
@@
 	10400 4075 11800 4075
 $Comp
-L device:R R121
+L LoTI_Board-rescue:R-device R121
 U 1 1 5FA9D488
 P 10925 4375
@@
 ADC0
 $Comp
-L device:R R124
+L LoTI_Board-rescue:R-device R124
 U 1 1 5CB16726
 P 12600 3575
@@
 $EndComp
 $Comp
-L device:LED D13
+L LoTI_Board-rescue:LED-device D13
 U 1 1 5CB1BE49
 P 13075 3575
@@
 	10400 3075 11175 3075
 $Comp
-L Connector:Test_Point TP?
+L LoTI_Board-rescue:Test_Point-Connector TP?
 U 1 1 62481FA3
 P 7100 1825

Commit message: Rev B updates
Parts:
- R117: value 10K -> DNF; Devtank 101-010 -> (none)
Changed lines of the file:
@@
 EESchema Schematic File Version 4
-LIBS:LoTI_Board-cache
-EELAYER 29 0
+EELAYER 30 0
 EELAYER END
 $Descr A3 16535 11693
@@
 Sheet 7 8
 Title "LoTI Board"
-Date "2019-07-03"
-Rev "Rev A"
+Date "2020-07-01"
+Rev "Rev B"
 Comp "Devtank Ltd"
 Comment1 ""
@@
 P 2550 3500
 F 0 "R117" H 2620 3546 50  0000 L CNN
-F 1 "10K" H 2620 3455 50  0000 L CNN
+F 1 "DNF" H 2620 3455 50  0000 L CNN
 F 2 "Resistor_SMD:R_0603_1608Metric" V 2480 3500 50  0001 C CNN
 F 3 "" H 2550 3500 50  0001 C CNN
-F 4 "101-010" H 0   0   50  0001 C CNN "Devtank"
+F 4 "" H 0   0   50  0001 C CNN "Devtank"
 	1    2550 3500
 	1    0    0    -1
