File: kicad_hiltop_loti_board/USB_Controller.sch (KiCad schematic (older format))
At the start: 48 parts, among them U10 LAN9513, U11 MIC2026-1YM, U12 SP3003-02XJ, U9 93LCxxA, Y1 25MHz Crystal

Commit message: updated drawing templates
Parts:
- U11: symbol SC_InterfaceBoard-rescue:MIC2026-1YM-Devtank -> LoTI_Board-rescue:MIC2026-1YM-Devtank-SC_InterfaceBoard-rescue
Changed lines of the file:
@@
 EESchema Schematic File Version 4
-LIBS:SC_InterfaceBoard-cache
+LIBS:LoTI_Board-cache
 EELAYER 26 0
 EELAYER END
@@
 encoding utf-8
 Sheet 4 8
-Title ""
-Date ""
-Rev ""
-Comp ""
+Title "LoTI Board"
+Date "2019-07-03"
+Rev "Rev A"
+Comp "Devtank Ltd"
 Comment1 ""
 Comment2 ""
@@
 USB4_PWR
 $Comp
-L SC_InterfaceBoard-rescue:MIC2026-1YM-Devtank U11
+L LoTI_Board-rescue:MIC2026-1YM-Devtank-SC_InterfaceBoard-rescue U11
 U 1 1 5C8E00A9
 P 10825 5000

Commit message: Rev A
Parts:
- C30, C31, C32, C33, C34, C35, C36, C37, C38, C39, C40, C41, C42, C43, C44, C45, C46, C47, C48, C49, C50, C51: symbol device:C -> LoTI_Board-rescue:C-device
- D12: symbol device:LED -> LoTI_Board-rescue:LED-device
- L1, L2: symbol device:Ferrite_Bead -> LoTI_Board-rescue:Ferrite_Bead-device
- R63, R64, R65, R66, R67, R68, R69, R70, R71, R72, R73, R74, R75: symbol device:R -> LoTI_Board-rescue:R-device
- TP106, TP108, TP114, TP115, TP116: symbol Connector:Test_Point -> LoTI_Board-rescue:Test_Point-Connector
- U9: symbol memory:93LCxxA -> LoTI_Board-rescue:93LCxxA-memory
- Y1: symbol device:Crystal_GND24 -> LoTI_Board-rescue:Crystal_GND24-device
Changed lines of the file:
@@
 EESchema Schematic File Version 4
 LIBS:LoTI_Board-cache
-EELAYER 26 0
+EELAYER 29 0
 EELAYER END
 $Descr A3 16535 11693
@@
 	3975 2850 3550 2850
 $Comp
-L device:R R69
+L LoTI_Board-rescue:R-device R69
 U 1 1 5C897D02
 P 3375 3550
@@
 $EndComp
 $Comp
-L device:C C31
+L LoTI_Board-rescue:C-device C31
 U 1 1 5C89C60B
 P 1175 10050
@@
 $EndComp
 $Comp
-L device:C C32
+L LoTI_Board-rescue:C-device C32
 U 1 1 5C89C6A9
 P 1600 10050
@@
 $EndComp
 $Comp
-L device:C C34
+L LoTI_Board-rescue:C-device C34
 U 1 1 5C89C6DD
 P 2050 10050
@@
 Connection ~ 1600 10275
 $Comp
-L device:Ferrite_Bead L1
+L LoTI_Board-rescue:Ferrite_Bead-device L1
 U 1 1 5C8A132B
 P 3350 9825
@@
 $EndComp
 $Comp
-L device:C C35
+L LoTI_Board-rescue:C-device C35
 U 1 1 5C8A1435
 P 2900 10050
@@
 $EndComp
 $Comp
-L device:C C38
+L LoTI_Board-rescue:C-device C38
 U 1 1 5C8A14EC
 P 3800 10050
@@
 	3800 10200 3800 10325
 $Comp
-L device:C C39
+L LoTI_Board-rescue:C-device C39
 U 1 1 5C8A6AA0
 P 4475 10050
@@
 $EndComp
 $Comp
-L device:C C40
+L LoTI_Board-rescue:C-device C40
 U 1 1 5C8A6BD8
 P 4925 10050
@@
 $EndComp
 $Comp
-L device:C C41
+L LoTI_Board-rescue:C-device C41
 U 1 1 5C8A6C1E
 P 5375 10050
@@
 $EndComp
 $Comp
-L device:C C42
+L LoTI_Board-rescue:C-device C42
 U 1 1 5C8A6C66
 P 5825 10050
@@
 $EndComp
 $Comp
-L device:C C43
+L LoTI_Board-rescue:C-device C43
 U 1 1 5C8A6CCA
 P 6275 10050
@@
 Connection ~ 5825 9800
 $Comp
-L device:Ferrite_Bead L2
+L LoTI_Board-rescue:Ferrite_Bead-device L2
 U 1 1 5C8B47F3
 P 7400 9800
@@
 $EndComp
 $Comp
-L device:C C46
+L LoTI_Board-rescue:C-device C46
 U 1 1 5C8B4B4C
 P 8700 10025
@@
 $EndComp
 $Comp
-L device:C C44
+L LoTI_Board-rescue:C-device C44
 U 1 1 5C8B4C20
 P 7850 10025
@@
 $EndComp
 $Comp
-L device:C C45
+L LoTI_Board-rescue:C-device C45
 U 1 1 5C8B4CF2
 P 8275 10025
@@
 $EndComp
 $Comp
-L device:C C47
+L LoTI_Board-rescue:C-device C47
 U 1 1 5C8B4EB4
 P 9125 10025
@@
 $EndComp
 $Comp
-L device:C C48
+L LoTI_Board-rescue:C-device C48
 U 1 1 5C8B4F0C
 P 9550 10025
@@
 $EndComp
 $Comp
-L device:C C50
+L LoTI_Board-rescue:C-device C50
 U 1 1 5C8B4FD2
 P 9975 10025
@@
 $EndComp
 $Comp
-L device:C C51
+L LoTI_Board-rescue:C-device C51
 U 1 1 5C8B5034
 P 10400 10025
@@
 $EndComp
 $Comp
-L device:LED D12
+L LoTI_Board-rescue:LED-device D12
 U 1 1 5C8E038B
 P 12050 5325
@@
 PCTL4
 $Comp
-L device:R R75
+L LoTI_Board-rescue:R-device R75
 U 1 1 5C8F8534
 P 12050 5725
@@
 	12050 5875 12050 6000
 $Comp
-L device:C C49
+L LoTI_Board-rescue:C-device C49
 U 1 1 5C945BF1
 P 9625 5175
@@
 RXN
 $Comp
-L device:R R72
+L LoTI_Board-rescue:R-device R72
 U 1 1 5D43F29C
 P 7500 4450
@@
 $EndComp
 $Comp
-L device:R R73
+L LoTI_Board-rescue:R-device R73
 U 1 1 5D44701B
 P 7850 4450
@@
 $EndComp
 $Comp
-L device:R R71
+L LoTI_Board-rescue:R-device R71
 U 1 1 5D44708F
 P 7150 4450
@@
 $EndComp
 $Comp
-L device:R R74
+L LoTI_Board-rescue:R-device R74
 U 1 1 5D44716A
 P 8200 4450
@@
 	8200 5100 8475 5100
 $Comp
-L Connector:Test_Point TP114
+L LoTI_Board-rescue:Test_Point-Connector TP114
 U 1 1 5D4972CC
 P 9050 2250
@@
 	9050 2425 9300 2425
 $Comp
-L Connector:Test_Point TP115
+L LoTI_Board-rescue:Test_Point-Connector TP115
 U 1 1 5D49E0D2
 P 9050 2850
@@
 $EndComp
 $Comp
-L Connector:Test_Point TP116
+L LoTI_Board-rescue:Test_Point-Connector TP116
 U 1 1 5D49E172
 P 9050 3450
@@
 	6375 5700 7325 5700
 $Comp
-L Connector:Test_Point TP108
+L LoTI_Board-rescue:Test_Point-Connector TP108
 U 1 1 5D5021EF
 P 3875 9750
@@
 	3800 9750 3800 9825
 $Comp
-L Connector:Test_Point TP106
+L LoTI_Board-rescue:Test_Point-Connector TP106
 U 1 1 5D50F109
 P 1100 9750
@@
 	3800 7500 3800 7600
 $Comp
-L device:R R70
+L LoTI_Board-rescue:R-device R70
 U 1 1 5D545083
 P 3700 4650
@@
 $EndComp
 $Comp
-L device:R R68
+L LoTI_Board-rescue:R-device R68
 U 1 1 5D54521E
 P 3075 4900
@@
 	2750 4900 2925 4900
 $Comp
-L device:R R65
+L LoTI_Board-rescue:R-device R65
 U 1 1 5D5692BF
 P 2550 7250
@@
 USB2.0 to be routed as differential impedance 90R
 $Comp
-L device:Crystal_GND24 Y1
+L LoTI_Board-rescue:Crystal_GND24-device Y1
 U 1 1 5D56F65E
 P 2550 7650
@@
 $EndComp
 $Comp
-L device:C C33
+L LoTI_Board-rescue:C-device C33
 U 1 1 5D5789EB
 P 2025 7875
@@
 $EndComp
 $Comp
-L device:C C37
+L LoTI_Board-rescue:C-device C37
 U 1 1 5D578DA6
 P 3075 7875
@@
 	3575 5600 3575 5875
 $Comp
-L device:C C36
+L LoTI_Board-rescue:C-device C36
 U 1 1 5D60A9D4
 P 2925 6275
@@
 	2925 6475 2925 6425
 $Comp
-L device:R R67
+L LoTI_Board-rescue:R-device R67
 U 1 1 5D616FCB
 P 2925 5850
@@
 $EndComp
 $Comp
-L device:R R66
+L LoTI_Board-rescue:R-device R66
 U 1 1 5D7D8DBF
 P 2900 3350
@@
 	3050 3350 3975 3350
 $Comp
-L device:R R64
+L LoTI_Board-rescue:R-device R64
 U 1 1 5CA7094C
 P 2475 6100
@@
 EEDI
 $Comp
-L memory:93LCxxA U9
+L LoTI_Board-rescue:93LCxxA-memory U9
 U 1 1 5EA74A54
 P 1700 4400
@@
 $EndComp
 $Comp
-L device:R R63
+L LoTI_Board-rescue:R-device R63
 U 1 1 5EA7508E
 P 1100 4750
@@
 	1225 4200 1400 4200
 $Comp
-L device:C C30
+L LoTI_Board-rescue:C-device C30
 U 1 1 5EAD1AAC
 P 975 3875
