File: kicad_hiltop_loti_board/USB_Debug.sch (KiCad schematic (older format))
At the start: 13 parts, among them U13 CP2102N-A01-GQFN24

Commit message: Rev A
Parts:
- C52, C55, C56: symbol device:C -> LoTI_Board-rescue:C-device
- R76, R77, R78, R79, R80, R81, R82, R83, R84: symbol device:R -> LoTI_Board-rescue:R-device
- U13: symbol silabs:CP2102N-A01-GQFN24 -> LoTI_Board-rescue:CP2102N-A01-GQFN24-silabs
Changed lines of the file:
@@
 EESchema Schematic File Version 4
 LIBS:LoTI_Board-cache
-EELAYER 26 0
+EELAYER 29 0
 EELAYER END
 $Descr A4 11693 8268
@@
 USB_N
 $Comp
-L silabs:CP2102N-A01-GQFN24 U13
+L LoTI_Board-rescue:CP2102N-A01-GQFN24-silabs U13
 U 1 1 5C2328D1
 P 5525 3475
@@
 	5525 2325 5525 2450
 $Comp
-L device:R R78
+L LoTI_Board-rescue:R-device R78
 U 1 1 5C3A3F19
 P 4050 3775
@@
 	2675 2875 2975 2875
 $Comp
-L device:R R?
+L LoTI_Board-rescue:R-device R?
 U 1 1 5C3AE29F
 P 6650 3975
@@
 $EndComp
 $Comp
-L device:R R?
+L LoTI_Board-rescue:R-device R?
 U 1 1 5C3AF9C1
 P 6650 4075
@@
 	6125 3275 7125 3275
 $Comp
-L device:R R83
+L LoTI_Board-rescue:R-device R83
 U 1 1 5C3B4D7B
 P 7275 3175
@@
 $EndComp
 $Comp
-L device:R R84
+L LoTI_Board-rescue:R-device R84
 U 1 1 5C3B4EF0
 P 7275 3275
@@
 	7425 3275 7575 3275
 $Comp
-L device:R R76
+L LoTI_Board-rescue:R-device R76
 U 1 1 5C3C0EE1
 P 3125 2875
@@
 $EndComp
 $Comp
-L device:R R77
+L LoTI_Board-rescue:R-device R77
 U 1 1 5C3C0F83
 P 3825 2625
@@
 	3825 2400 3825 2475
 $Comp
-L device:C C55
+L LoTI_Board-rescue:C-device C55
 U 1 1 5C3C60B5
 P 5800 2225
@@
 $EndComp
 $Comp
-L device:C C56
+L LoTI_Board-rescue:C-device C56
 U 1 1 5C3C6FB8
 P 6225 2225
@@
 NoConn ~ 6125 3575
 $Comp
-L device:C C?
+L LoTI_Board-rescue:C-device C?
 U 1 1 5CA83BDF
 P 3475 3275
@@
 	6125 3975 6500 3975
 $Comp
-L device:R R?
+L LoTI_Board-rescue:R-device R?
 U 1 1 5CA8BD2A
 P 6650 3875
@@
 	6125 3875 6500 3875
 $Comp
-L device:R R?
+L LoTI_Board-rescue:R-device R?
 U 1 1 5CA8CA4A
 P 6650 3775

Commit message: Rev B updates
Parts:
- added C54: 100nF, Capacitor_SMD:C_0603_1608Metric, symbol LoTI_Board-rescue:C-device
- added R152: 47K, Resistor_SMD:R_0603_1608Metric, symbol LoTI_Board-rescue:R-device
- added U23: M74VHC1GT14DFT2G, Package_TO_SOT_SMD:SOT-353_SC-70-5, symbol Devtank:NL17SZ14
- R78: value 0R -> 24K
- R79, R80: value 330R -> 0R; Devtank 101-024 -> 101-005
Connections:
- net +3V3: now also C54.2, U23.5 (VCC)
- net GND: now also C54.1, R152.1, U23.3 (VSS)
- net STM_BOOT0: now also U23.4; no longer R79.1
- net at R78.1, U13.8 (VBUS): now also R152.2
- new net: R79.1, U23.2
Changed lines of the file:
@@
 EESchema Schematic File Version 4
-LIBS:LoTI_Board-cache
-EELAYER 29 0
+EELAYER 30 0
 EELAYER END
 $Descr A4 11693 8268
 encoding utf-8
-Sheet 5 8
+Sheet 4 8
 Title "LoTI Board"
-Date "2019-07-03"
-Rev "Rev A"
+Date "2020-07-01"
+Rev "Rev B"
 Comp "Devtank Ltd"
 Comment1 ""
@@
 P 4050 3775
 F 0 "R78" V 3950 3675 50  0000 C CNN
-F 1 "0R" V 3950 3850 50  0000 C CNN
+F 1 "24K" V 3950 3850 50  0000 C CNN
 F 2 "Resistor_SMD:R_0603_1608Metric" V 3980 3775 50  0001 C CNN
 F 3 "" H 4050 3775 50  0001 C CNN
@@
 $EndComp
 Wire Wire Line
-	4925 3775 4200 3775
+	4925 3775 4450 3775
 Text HLabel 3025 3775 0    60   Input ~ 0
 USB_BUS_PWR
@@
 AR Path="/5CA829FD/5CA8BD2A" Ref="R80"  Part="1"
 F 0 "R80" V 6600 3650 50  0000 C CNN
-F 1 "330R" V 6600 4100 50  0000 C CNN
+F 1 "0R" V 6600 4100 50  0000 C CNN
 F 2 "Resistor_SMD:R_0603_1608Metric" V 6580 3875 50  0001 C CNN
 F 3 "" H 6650 3875 50  0000 C CNN
-F 4 "101-024" V 6650 3875 60  0001 C CNN "Devtank"
+F 4 "101-005" V 6650 3875 60  0001 C CNN "Devtank"
 	1    6650 3875
 	0    1    1    0
@@
 AR Path="/5CA829FD/5CA8CA4A" Ref="R79"  Part="1"
 F 0 "R79" V 6600 3550 50  0000 C CNN
-F 1 "330R" V 6600 4000 50  0000 C CNN
+F 1 "0R" V 6600 4000 50  0000 C CNN
 F 2 "Resistor_SMD:R_0603_1608Metric" V 6580 3775 50  0001 C CNN
 F 3 "" H 6650 3775 50  0000 C CNN
-F 4 "101-024" V 6650 3775 60  0001 C CNN "Devtank"
+F 4 "101-005" V 6650 3775 60  0001 C CNN "Devtank"
 	1    6650 3775
 	0    1    1    0
@@
 	6125 3775 6500 3775
 Wire Wire Line
-	6800 3775 7625 3775
-Wire Wire Line
 	6800 3875 7625 3875
 Wire Wire Line
@@
 Wire Wire Line
 	6800 4075 7625 4075
-Text HLabel 7625 3775 2    60   Output ~ 0
+Text HLabel 9150 3775 2    60   Output ~ 0
 STM_BOOT0
 Text HLabel 7625 3875 2    60   Output ~ 0
@@
 Wire Wire Line
 	4650 2325 4650 3475
+$Comp
+L LoTI_Board-rescue:R-device R152
+U 1 1 5F705021
+P 4450 4250
+F 0 "R152" H 4275 4200 50  0000 C CNN
+F 1 "47K" H 4300 4300 50  0000 C CNN
+F 2 "Resistor_SMD:R_0603_1608Metric" V 4380 4250 50  0001 C CNN
+F 3 "" H 4450 4250 50  0001 C CNN
+	1    4450 4250
+	-1   0    0    1
+$EndComp
+Wire Wire Line
+	4450 3775 4450 4100
+Connection ~ 4450 3775
+Wire Wire Line
+	4450 3775 4200 3775
+$Comp
+L power:GND #PWR037
+U 1 1 5F7066D6
+P 4450 4525
+F 0 "#PWR037" H 4450 4275 50  0001 C CNN
+F 1 "GND" H 4455 4352 50  0000 C CNN
+F 2 "" H 4450 4525 50  0001 C CNN
+F 3 "" H 4450 4525 50  0001 C CNN
+	1    4450 4525
+	1    0    0    -1
+$EndComp
+Wire Wire Line
+	4450 4400 4450 4525
+$Comp
+L Devtank:NL17SZ14 U23
+U 1 1 5F80DDDE
+P 8450 3775
+F 0 "U23" H 8550 3925 50  0000 C CNN
+F 1 "M74VHC1GT14DFT2G" H 8875 3625 50  0000 C CNN
+F 2 "Package_TO_SOT_SMD:SOT-353_SC-70-5" H 8450 3775 60  0001 C CNN
+F 3 "" H 8450 3775 60  0001 C CNN
+	1    8450 3775
+	1    0    0    -1
+$EndComp
+Wire Wire Line
+	6800 3775 8000 3775
+Wire Wire Line
+	9150 3775 8900 3775
+$Comp
+L LoTI_Board-rescue:C-device C54
+U 1 1 5F81CFF7
+P 8725 3325
+F 0 "C54" V 8575 3275 50  0000 L CNN
+F 1 "100nF" V 8875 3225 50  0000 L CNN
+F 2 "Capacitor_SMD:C_0603_1608Metric" H 8763 3175 50  0001 C CNN
+F 3 "" H 8725 3325 50  0001 C CNN
+F 4 "105-002" H 8725 3325 50  0001 C CNN "Devtank"
+	1    8725 3325
+	0    1    1    0
+$EndComp
+$Comp
+L power:GND #PWR0134
+U 1 1 5F81D655
+P 9050 3425
+F 0 "#PWR0134" H 9050 3175 50  0001 C CNN
+F 1 "GND" H 9050 3275 50  0000 C CNN
+F 2 "" H 9050 3425 50  0001 C CNN
+F 3 "" H 9050 3425 50  0001 C CNN
+	1    9050 3425
+	1    0    0    -1
+$EndComp
+$Comp
+L power:+3V3 #PWR0205
+U 1 1 5F81DB05
+P 8400 3125
+F 0 "#PWR0205" H 8400 2975 50  0001 C CNN
+F 1 "+3V3" H 8415 3298 50  0000 C CNN
+F 2 "" H 8400 3125 50  0001 C CNN
+F 3 "" H 8400 3125 50  0001 C CNN
+	1    8400 3125
+	1    0    0    -1
+$EndComp
+Wire Wire Line
+	8400 3125 8400 3325
+$Comp
+L power:GND #PWR0208
+U 1 1 5F8209D4
+P 8400 4200
+F 0 "#PWR0208" H 8400 3950 50  0001 C CNN
+F 1 "GND" H 8400 4050 50  0000 C CNN
+F 2 "" H 8400 4200 50  0001 C CNN
+F 3 "" H 8400 4200 50  0001 C CNN
+	1    8400 4200
+	1    0    0    -1
+$EndComp
+Wire Wire Line
+	8400 4200 8400 3875
+Wire Wire Line
+	8575 3325 8400 3325
+Connection ~ 8400 3325
+Wire Wire Line
+	8400 3325 8400 3675
+Wire Wire Line
+	9050 3425 9050 3325
+Wire Wire Line
+	9050 3325 8875 3325
 $EndSCHEMATC
